Commit message: removed mentions to gazebo

File: src/oruga_pkg/description/models/oruga/camera.xacro (robot description, xacro)
@@ -1,5 +1,5 @@
 <?xml version="1.0"?>
 <robot xmlns:xacro="http://www.ros.org/wiki/xacro">
-  <xacro:macro name="oruga_camera" params="use_camera use_gazebo">
+  <xacro:macro name="oruga_camera" params="use_camera">
     <xacro:if value="${use_camera}">
       <link name="camera_link">
@@ -24,29 +24,4 @@
         <child link="camera_link_optical" />
       </joint>
-      <xacro:if value="$(arg use_gazebo)">
-        <gazebo reference="camera_link">
-          <material>Gazebo/Black</material>
-          <sensor name="camera" type="camera">
-            <pose> 0 0 0 0 0 0 </pose>
-            <visualize>true</visualize>
-            <update_rate>10</update_rate>
-            <camera>
-              <camera_info_topic>camera/camera_info</camera_info_topic>
-              <horizontal_fov>1.089</horizontal_fov>
-              <image>
-                <format>R8G8B8</format>
-                <width>640</width>
-                <height>480</height>
-              </image>
-              <clip>
-                <near>0.05</near>
-                <far>8.0</far>
-              </clip>
-            </camera>
-            <topic>camera/image_raw</topic>
-            <gz_frame_id>camera_link_optical</gz_frame_id>
-          </sensor>
-        </gazebo>
-      </xacro:if>
     </xacro:if>
   </xacro:macro>

File: src/oruga_pkg/description/models/oruga/imu.xacro (robot description, xacro)
@@ -1,5 +1,5 @@
 <?xml version="1.0"?>
 <robot xmlns:xacro="http://www.ros.org/wiki/xacro">
-  <xacro:macro name="oruga_imu" params="use_imu use_gazebo">
+  <xacro:macro name="oruga_imu" params="use_imu">
     <xacro:if value="${use_imu}">
       <link name="imu_link"></link>
@@ -10,26 +10,4 @@
           rpy="${imu_offset_r} ${imu_offset_p} ${imu_offset_y}" />
       </joint>
-      <xacro:if value="$(arg use_gazebo)">
-        <gazebo reference="imu_link">
-          <gravity>true</gravity>
-          <sensor name="imu_sensor" type="imu">
-            <always_on>true</always_on>
-            <update_rate>100</update_rate>
-            <visualize>true</visualize>
-            <topic>imu_raw</topic>
-            <plugin filename="libgazebo_ros_imu_sensor.so" name="imu_plugin">
-              <topicName>imu</topicName>
-              <bodyName>imu_link</bodyName>
-              <updateRateHZ>10.0</updateRateHZ>
-              <gaussianNoise>0.0</gaussianNoise>
-              <xyzOffset>0 0 0</xyzOffset>
-              <rpyOffset>0 0 0</rpyOffset>
-              <frameName>imu_link</frameName>
-              <initialOrientationAsReference>false</initialOrientationAsReference>
-            </plugin>
-            <pose>0 0 0 0 0 0</pose>
-          </sensor>
-        </gazebo>
-      </xacro:if>
     </xacro:if>
   </xacro:macro>

File: src/oruga_pkg/description/models/oruga/lidar.xacro (robot description, xacro)
@@ -1,5 +1,5 @@
 <?xml version="1.0"?>
 <robot xmlns:xacro="http://www.ros.org/wiki/xacro">
-  <xacro:macro name="oruga_lidar" params="use_lidar use_gazebo">
+  <xacro:macro name="oruga_lidar" params="use_lidar">
     <xacro:if value="${use_lidar}">
       <link name="lidar_link">
@@ -18,30 +18,4 @@
           rpy="0 0 0" />
       </joint>
-      <xacro:if value="$(arg use_gazebo)">
-        <gazebo reference="lidar_link">
-          <!-- LDS-01 LIDAR -->
-          <sensor name="laser" type="gpu_lidar">
-            <pose> 0 0 0 0 0 0 </pose>
-            <visualize>true</visualize>
-            <always_on>true</always_on>
-            <update_rate>10</update_rate>
-            <lidar>
-              <scan>
-                <horizontal>
-                  <samples>360</samples>
-                  <min_angle>-3.14</min_angle>
-                  <max_angle>3.14</max_angle>
-                </horizontal>
-              </scan>
-              <range>
-                <min>0.12</min>
-                <max>3.5</max>
-              </range>
-            </lidar>
-            <topic>scan</topic>
-            <gz_frame_id>lidar_link</gz_frame_id>
-          </sensor>
-        </gazebo>
-      </xacro:if>
     </xacro:if>
   </xacro:macro>

File: src/oruga_pkg/description/models/oruga/oruga.urdf.xacro (robot description, xacro)
@@ -1,5 +1,4 @@
 <?xml version="1.0"?>
 <robot xmlns:xacro="http://www.ros.org/wiki/xacro"  name="oruga">
-    <xacro:arg name="use_gazebo" default="false" />
     <xacro:arg name="use_imu" default="true" />
     <xacro:arg name="use_lidar" default="false" />
@@ -7,8 +6,8 @@
     <xacro:include filename="a4wd3.xacro" />
     <xacro:include filename="imu.xacro" />
-    <xacro:oruga_imu use_imu="$(arg use_imu)" use_gazebo="$(arg use_gazebo)"/>
+    <xacro:oruga_imu use_imu="$(arg use_imu)"/>
     <xacro:include filename="lidar.xacro" />
-    <xacro:oruga_lidar use_lidar="$(arg use_lidar)" use_gazebo="$(arg use_gazebo)"/>
+    <xacro:oruga_lidar use_lidar="$(arg use_lidar)" />
     <xacro:include filename="camera.xacro" />
-    <xacro:oruga_camera use_camera="$(arg use_camera)" use_gazebo="$(arg use_gazebo)"/>
+    <xacro:oruga_camera use_camera="$(arg use_camera)" />
 </robot>
